File: hardware/iguana_version/PCB/sirius_v1.kicad_pcb (KiCad board)
At the start: 2 copper layers, 80 x 50 mm, 122 parts, among them J1 BAT, J10 OLED, J12 USB_B_Micro, J13 HDR-2x1, J14 Conn_01x02, J17 Conn_Coaxial, J18 IN, J19 IN, J2 HDR-2x1, J3 IN, J4 Cap. Moisture Sensor, J5 ds18b20, J6 SHT31, J7 NPK/H Sensor, J8 ON OFF, J9 HDR-3x1, Q1 Q_PMOS_GSD, Q10 BSS138, Q2 Q_PMOS_GSD, Q3 Q_Dual_NPN_NPN_BRT_E1B1C2E2B2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, Q4 BSS138, Q6 Q_PMOS_GSD, Q7 Q_PMOS_GSD, Q9 BSS138, SW1 SW_DIP_x02, SW2 SW_DIP_x02, SW3 SW_DIP_x02, U1 DW01, U10 ESP32-WROOM-32D, U11 RV-8803, U12 RFM95W-915S2, U2 TP4056, U3 MT3608, U4 FS8205A, U5 AP2112K-3.3, U6 AP2112K-3.3, U8 AP2112K-3.3, U9 CH340C

Commit message: updating fab files
Parts:
- removed J8: ON OFF, Jumper:SolderJumper-2_P1.3mm_Open_RoundedPad1.0x1.5mm
- added JP4: SolderJumper_2_Open, Jumper:SolderJumper-2_P1.3mm_Open_RoundedPad1.0x1.5mm, F.Cu at (115.8, 63.0)
- added JP5: SolderJumper_2_Open, Jumper:SolderJumper-2_P1.3mm_Open_RoundedPad1.0x1.5mm, F.Cu at (110.0, 53.0)
- R35, R36: value 10K -> 330
- R39, R40: value 10K -> 0
- moved G*** 1.21 mm to (99.5, 50.1)
- moved J2 0.65 mm to (113.0, 51.9)
Routing:
- net /Vo_DCDC: track 30.6 -> 44.5 mm, vias 0 -> 1
- net /V_USB: track 12.4 -> 8.26 mm
- net +5V: track 155.4 -> 159.3 mm
- net GND: vias 145 -> 144
